File: pcb/Projektarbeit.kicad_pcb (KiCad board)
At the start: 2 copper layers, 63.8 x 24.5 mm, 26 parts, among them J1 JST_XH 01x02, J2 61300811121, J3 61300211121, U1 XIAO-ESP32S3, U2 WPME-FISM_SMT-8, U3 SI2307CDS-T1-BE3, U4 2N7002K-T1-GE3

Commit message: added html BOM
Parts:
- C6: value ?F -> 100nF
- R7: value ?kΩ -> 10kΩ
Changed lines of the file:
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@@
 			)
 		)
-		(property "Value" "?kΩ"
+		(property "Value" "10kΩ"
 			(at 0 1.65 0)
 			(layer "F.Fab")
@@
 			)
 		)
-		(property "Value" "?F"
+		(property "Value" "100nF"
 			(at -0.1 1.9968 0)
 			(layer "F.Fab")
